Commit message: fix(sim): pan the wrist camera onto where the arm carries it
The fixed jaw is rigid to the wrist camera, so where it lands in the frame
reports that camera's mounting and nothing else. Averaged over the 36 recorded
hardware episodes it sits 41 px from the sim render, purely horizontally, which
at f=546 is 4.25 degrees about the camera's own image-down axis. The joint's
roll carries that turn, and the sim jaw lands within a pixel of the recorded one.

About 2.7 degrees of it is play where the bracket meets the wrist, so this
describes the arm as it currently stands rather than the geometry alone.

Co-Authored-By: Claude Opus 5 (1M context) <noreply@anthropic.com>
Claude-Session: https://claude.ai/code/session_01SkMNrB6vs3idePeXavD7kz

File: sim/src/sim/description/so101.urdf (robot description, URDF)
Before this commit: robot so101_new_calib, 12 links, 11 joints
Joints:
- joint wrist_camera_frame_fixed_joint: origin xyz=0.0025 0.072010214 -0.000859294 rpy=-3.577922 -5.55112e-17 0 -> xyz=0.0025 0.072010214 -0.000859294 rpy=2.704208 -0.067216 0.031395
